File: PCB/battery.kicad_sch (KiCad schematic)
At the start: 1 part

Commit message: refactor: switch over to esp32-s3-wroom1 (#13)
This refactors to the esp32-s3 to avoid every problem we encountered with the raspberry pi options.
Parts:
- BT1: footprint (none) -> Battery:BatteryHolder_Keystone_1042_1x18650
Changed lines of the file:
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@@
 (kicad_sch
 	(version 20250114)
-	(generator "eeschema")
-	(generator_version "9.0")
+	(generator "kicaddy")
+	(generator_version "0.1.0")
 	(paper "A4")
 	(global_label "VBAT"
 		(shape passive)
-		(at 148.59 100.33 90)
+		(at 148.59 100.33 270)
 		(fields_autoplaced yes)
-		(effects
-			(font
-				(size 1.27 1.27)
-			)
-			(justify left)
-		)
-		(property "Intersheetrefs" "${INTERSHEET_REFS}"
-			(at 148.59 100.33 0)
-			(effects
-				(font
-					(size 1.27 1.27)
-				)
-				(hide yes)
-			)
-		)
+		(effects (font (size 1.27 1.27)) (justify left))
 	)
 	(global_label "GND"
 		(shape passive)
-		(at 148.59 110.49 270)
+		(at 148.59 110.49 90)
 		(fields_autoplaced yes)
-		(effects
-			(font
-				(size 1.27 1.27)
-			)
-			(justify right)
-		)
-		(property "Intersheetrefs" "${INTERSHEET_REFS}"
-			(at 148.59 110.49 0)
-			(effects
-				(font
-					(size 1.27 1.27)
-				)
-				(hide yes)
-			)
-		)
+		(effects (font (size 1.27 1.27)) (justify right))
 	)
 	(symbol
@@
 		(dnp no)
 		(fields_autoplaced yes)
-		(property "Reference" "BT1"
+		(property "Reference"
+			"BT1"
 			(at 151.13 107.95 0)
-			(effects
-				(font
-					(size 1.27 1.27)
-				)
-				(justify left)
-			)
+			(effects (font (size 1.27 1.27)) (justify left))
 		)
-		(property "Value" "Li-ion_18650_or_14500"
+		(property "Value"
+			"Li-ion_18650_or_14500"
 			(at 151.13 105.41 0)
-			(effects
-				(font
-					(size 1.27 1.27)
-				)
-				(justify left)
-			)
+			(effects (font (size 1.27 1.27)) (justify left))
 		)
-		(property "Footprint" ""
+		(property "Footprint"
+			"Battery:BatteryHolder_Keystone_1042_1x18650"
 			(at 148.59 106.934 90)
-			(effects
-				(font
-					(size 1.27 1.27)
-				)
-				(hide yes)
-			)
+			(effects (font (size 1.27 1.27)) (hide yes))
 		)
-		(property "Datasheet" "~"
+		(property "Datasheet"
+			"~"
 			(at 148.59 106.934 90)
-			(effects
-				(font
-					(size 1.27 1.27)
-				)
-				(hide yes)
-			)
+			(effects (font (size 1.27 1.27)) (hide yes))
 		)
-		(property "Description" "Multiple-cell battery"
+		(property "Description"
+			"Multiple-cell battery"
 			(at 148.59 105.41 0)
-			(effects
-				(font
-					(size 1.27 1.27)
-				)
-				(hide yes)
-			)
+			(effects (font (size 1.27 1.27)) (hide yes))
 		)
-		(property "Sim.Device" "V"
+		(property "Sim.Device"
+			"V"
 			(at 148.59 105.41 0)
-			(effects
-				(font
-					(size 1.27 1.27)
-				)
-				(hide yes)
-			)
+			(effects (font (size 1.27 1.27)) (hide yes))
 		)
-		(property "Sim.Type" "DC"
+		(property "Sim.Type"
+			"DC"
 			(at 148.59 105.41 0)
-			(effects
-				(font
-					(size 1.27 1.27)
-				)
-				(hide yes)
-			)
+			(effects (font (size 1.27 1.27)) (hide yes))
 		)
-		(property "Sim.Pins" "1=+ 2=-"
+		(property "Sim.Pins"
+			"1=+ 2=-"
 			(at 148.59 105.41 0)
-			(effects
-				(font
-					(size 1.27 1.27)
-				)
-				(hide yes)
-			)
+			(effects (font (size 1.27 1.27)) (hide yes))
 		)
-		(pin "1"
-		)
-		(pin "2"
-		)
+		(pin "1")
+		(pin "2")
 		(instances
-			(project "snips_controller"
-				(path "/70589bdd-acbd-4920-8e78-aa58d10832b9/6bc1f003-e00b-454c-a62b-fdbb357b02b9"
+			(project ""
+				(path "/868f8289-8434-4465-b2f4-2accc5e40bab/748cb1dd-d7df-4e73-a93b-27e67a5ba349"
 					(reference "BT1")
 					(unit 1)
@@
 		)
 	)
+	(sheet_instances
+		(path "/868f8289-8434-4465-b2f4-2accc5e40bab/748cb1dd-d7df-4e73-a93b-27e67a5ba349"
+			(page "1")
+		)
+	)
+	(embedded_fonts no)
 )
