File: PCB/hall_trigger.kicad_sch (KiCad schematic)
At the start: 2 parts

Commit message: refactor: erc is clean
This gets the schematic as clean as it can be.
Parts:
- removed C_HALL: 100nF, symbol Device:C
- removed U_HALL: DRV5055A2, Package_TO_SOT_THT:TO-92_Inline, symbol Sensor_Magnetic:DRV5055A2xLPGxQ1
- added C_HALL1: 100nF, symbol Device:C
- added U_HALL1: DRV5055A2, Package_TO_SOT_THT:TO-92_Inline, symbol Sensor_Magnetic:DRV5055A2xLPGxQ1
Connections:
- net 3V3: now also C_HALL1.1, U_HALL1.1 (VCC)
- net GND: now also C_HALL1.2, U_HALL1.2 (GND)
- net TRIG_ANALOG: now also U_HALL1.3 (OUT)
Changed lines of the file:
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@@
+	(global_label "GND"
+		(shape passive)
+		(at 128.27 106.68 270)
+		(fields_autoplaced yes)
+		(effects
+			(font
+				(size 1.27 1.27)
+			)
+			(justify right)
+		)
+		(property "Intersheetrefs" "${INTERSHEET_REFS}"
+			(at 128.27 106.68 0)
+			(effects
+				(font
+					(size 1.27 1.27)
+				)
+				(hide yes)
+			)
+		)
+	)
 	(global_label "GND"
 		(shape passive)
@@
 		(property "Intersheetrefs" "${INTERSHEET_REFS}"
 			(at 166.37 116.84 0)
-			(effects
-				(font
-					(size 1.27 1.27)
-				)
-				(hide yes)
-			)
-		)
-	)
-	(global_label "GND"
-		(shape passive)
-		(at 128.27 106.68 270)
-		(fields_autoplaced yes)
-		(effects
-			(font
-				(size 1.27 1.27)
-			)
-			(justify right)
-		)
-		(property "Intersheetrefs" "${INTERSHEET_REFS}"
-			(at 128.27 106.68 0)
 			(effects
 				(font
@@
 		(dnp no)
 		(fields_autoplaced yes)
-		(property "Reference" "C_HALL"
+		(property "Reference" "C_HALL1"
 			(at 167.005 115.57 0)
 			(effects
@@
 		(instances
 			(project "snips_controller"
-				(path "/2289c08f-f540-4e27-86fd-a28b71d1d149/f0a735b3-5667-42dc-802e-e46904fa430c"
-					(reference "C_HALL")
+				(path "/70589bdd-acbd-4920-8e78-aa58d10832b9/d425906b-e7ab-4d10-bbf9-3571bc43ff5e"
+					(reference "C_HALL1")
 					(unit 1)
 				)
@@
 		(dnp no)
 		(fields_autoplaced yes)
-		(property "Reference" "U_HALL"
+		(property "Reference" "U_HALL1"
 			(at 135.89 109.22 0)
 			(effects
@@
 		(instances
 			(project "snips_controller"
-				(path "/2289c08f-f540-4e27-86fd-a28b71d1d149/f0a735b3-5667-42dc-802e-e46904fa430c"
-					(reference "U_HALL")
+				(path "/70589bdd-acbd-4920-8e78-aa58d10832b9/d425906b-e7ab-4d10-bbf9-3571bc43ff5e"
+					(reference "U_HALL1")
 					(unit 1)
 				)

Commit message: refactor: switch over to esp32-s3-wroom1 (#13)
This refactors to the esp32-s3 to avoid every problem we encountered with the raspberry pi options.
Parts:
- removed C_HALL1: 100nF, symbol Device:C
- removed U_HALL1: DRV5055A2, Package_TO_SOT_THT:TO-92_Inline, symbol Sensor_Magnetic:DRV5055A2xLPGxQ1
- added C_HALL: 100nF, Capacitor_SMD:C_0402_1005Metric, symbol Device:C
- added U_HALL: DRV5055A2, Package_TO_SOT_THT:TO-92_Inline, symbol Sensor_Magnetic:DRV5055A2xLPGxQ1
Connections:
- net 3V3: now also C_HALL.1, U_HALL.1 (VCC)
- net GND: now also C_HALL.2, U_HALL.2 (GND)
- net TRIG_ANALOG: now also U_HALL.3 (OUT)
Changed lines of the file:
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@@
 (kicad_sch
 	(version 20250114)
-	(generator "eeschema")
-	(generator_version "9.0")
+	(generator "kicaddy")
+	(generator_version "0.1.0")
 	(paper "A4")
 	(global_label "3V3"
 		(shape passive)
-		(at 166.37 109.22 90)
+		(at 128.27 86.36 270)
 		(fields_autoplaced yes)
-		(effects
-			(font
-				(size 1.27 1.27)
-			)
-			(justify left)
-		)
-		(property "Intersheetrefs" "${INTERSHEET_REFS}"
-			(at 166.37 109.22 0)
-			(effects
-				(font
-					(size 1.27 1.27)
-				)
-				(hide yes)
-			)
-		)
+		(effects (font (size 1.27 1.27)) (justify left))
 	)
 	(global_label "3V3"
 		(shape passive)
-		(at 128.27 86.36 90)
+		(at 166.37 109.22 270)
 		(fields_autoplaced yes)
-		(effects
-			(font
-				(size 1.27 1.27)
-			)
-			(justify left)
-		)
-		(property "Intersheetrefs" "${INTERSHEET_REFS}"
-			(at 128.27 86.36 0)
-			(effects
-				(font
-					(size 1.27 1.27)
-				)
-				(hide yes)
-			)
-		)
+		(effects (font (size 1.27 1.27)) (justify left))
 	)
 	(global_label "GND"
 		(shape passive)
-		(at 128.27 106.68 270)
+		(at 128.27 106.68 90)
 		(fields_autoplaced yes)
-		(effects
-			(font
-				(size 1.27 1.27)
-			)
-			(justify right)
-		)
-		(property "Intersheetrefs" "${INTERSHEET_REFS}"
-			(at 128.27 106.68 0)
-			(effects
-				(font
-					(size 1.27 1.27)
-				)
-				(hide yes)
-			)
-		)
+		(effects (font (size 1.27 1.27)) (justify right))
 	)
 	(global_label "GND"
 		(shape passive)
-		(at 166.37 116.84 270)
+		(at 166.37 116.84 90)
 		(fields_autoplaced yes)
-		(effects
-			(font
-				(size 1.27 1.27)
-			)
-			(justify right)
-		)
-		(property "Intersheetrefs" "${INTERSHEET_REFS}"
-			(at 166.37 116.84 0)
-			(effects
-				(font
-					(size 1.27 1.27)
-				)
-				(hide yes)
-			)
-		)
+		(effects (font (size 1.27 1.27)) (justify right))
 	)
 	(hierarchical_label "TRIG_ANALOG"
 		(shape output)
-		(at 138.43 96.52 0)
-		(effects
-			(font
-				(size 1.27 1.27)
+		(at 138.43 96.52 180)
+	)
+	(symbol
+		(lib_id "Sensor_Magnetic:DRV5055A2xLPGxQ1")
+		(at 130.81 96.52 0)
+		(unit 1)
+		(exclude_from_sim no)
+		(in_bom yes)
+		(on_board yes)
+		(dnp no)
+		(fields_autoplaced yes)
+		(property "Reference"
+			"U_HALL"
+			(at 135.89 109.22 0)
+			(effects (font (size 1.27 1.27)))
+		)
+		(property "Value"
+			"DRV5055A2"
+			(at 138.43 106.68 0)
+			(effects (font (size 1.27 1.27)))
+		)
+		(property "Footprint"
+			"Package_TO_SOT_THT:TO-92_Inline"
+			(at 130.81 96.52 0)
+			(effects (font (size 1.27 1.27)) (hide yes))
+		)
+		(property "Datasheet"
+			"https://www.ti.com/lit/ds/symlink/drv5055-q1.pdf"
+			(at 130.81 96.52 0)
+			(effects (font (size 1.27 1.27)) (hide yes))
+		)
+		(property "Description"
+			"50 mV/mT,±42-mT, 20-kHz, 3.3/5V, TO-92"
+			(at 130.81 96.52 0)
+			(effects (font (size 1.27 1.27)) (hide yes))
+		)
+		(pin "1")
+		(pin "2")
+		(pin "3")
+		(instances
+			(project ""
+				(path "/868f8289-8434-4465-b2f4-2accc5e40bab/3b2478ec-2890-4ec8-b56f-d58b64ce58ab"
+					(reference "U_HALL")
+					(unit 1)
+				)
 			)
-			(justify left)
 		)
 	)
@@
 		(dnp no)
 		(fields_autoplaced yes)
-		(property "Reference" "C_HALL1"
+		(property "Reference"
+			"C_HALL"
 			(at 167.005 115.57 0)
-			(effects
-				(font
-					(size 1.27 1.27)
-				)
-				(justify left)
-			)
+			(effects (font (size 1.27 1.27)) (justify left))
 		)
-		(property "Value" "100nF"
+		(property "Value"
+			"100nF"
 			(at 167.005 110.49 0)
-			(effects
-				(font
-					(size 1.27 1.27)
-				)
-				(justify left)
-			)
+			(effects (font (size 1.27 1.27)) (justify left))
 		)
-		(property "Footprint" ""
+		(property "Footprint"
+			"Capacitor_SMD:C_0402_1005Metric"
 			(at 167.3352 109.22 0)
-			(effects
-				(font
-					(size 1.27 1.27)
-				)
-				(hide yes)
-			)
+			(effects (font (size 1.27 1.27)) (hide yes))
 		)
-		(property "Datasheet" "~"
+		(property "Datasheet"
+			"~"
 			(at 166.37 113.03 0)
-			(effects
-				(font
-					(size 1.27 1.27)
-				)
-				(hide yes)
-			)
+			(effects (font (size 1.27 1.27)) (hide yes))
 		)
-		(property "Description" "Unpolarized capacitor"
+		(property "Description"
+			"Unpolarized capacitor"
 			(at 166.37 113.03 0)
-			(effects
-				(font
-					(size 1.27 1.27)
-				)
-				(hide yes)
-			)
+			(effects (font (size 1.27 1.27)) (hide yes))
 		)
-		(pin "1"
-		)
-		(pin "2"
-		)
+		(pin "1")
+		(pin "2")
 		(instances
-			(project "snips_controller"
-				(path "/70589bdd-acbd-4920-8e78-aa58d10832b9/d425906b-e7ab-4d10-bbf9-3571bc43ff5e"
-					(reference "C_HALL1")
+			(project ""
+				(path "/868f8289-8434-4465-b2f4-2accc5e40bab/3b2478ec-2890-4ec8-b56f-d58b64ce58ab"
+					(reference "C_HALL")
 					(unit 1)
 				)
@@
 		)
 	)
-	(symbol
-		(lib_id "Sensor_Magnetic:DRV5055A2xLPGxQ1")
-		(at 130.81 96.52 0)
-		(unit 1)
-		(exclude_from_sim no)
-		(in_bom yes)
-		(on_board yes)
-		(dnp no)
-		(fields_autoplaced yes)
-		(property "Reference" "U_HALL1"
-			(at 135.89 109.22 0)
-			(effects
-				(font
-					(size 1.27 1.27)
-				)
-			)
-		)
-		(property "Value" "DRV5055A2"
-			(at 138.43 106.68 0)
-			(effects
-				(font
-					(size 1.27 1.27)
-				)
-			)
-		)
-		(property "Footprint" "Package_TO_SOT_THT:TO-92_Inline"
-			(at 130.81 96.52 0)
-			(effects
-				(font
-					(size 1.27 1.27)
-				)
-				(hide yes)
-			)
-		)
-		(property "Datasheet" "https://www.ti.com/lit/ds/symlink/drv5055-q1.pdf"
-			(at 130.81 96.52 0)
-			(effects
-				(font
-					(size 1.27 1.27)
-				)
-				(hide yes)
-			)
-		)
-		(property "Description" "50 mV/mT,±42-mT, 20-kHz, 3.3/5V, TO-92"
-			(at 130.81 96.52 0)
-			(effects
-				(font
-					(size 1.27 1.27)
-				)
-				(hide yes)
-			)
-		)
-		(pin "1"
-		)
-		(pin "2"
-		)
-		(pin "3"
-		)
-		(instances
-			(project "snips_controller"
-				(path "/70589bdd-acbd-4920-8e78-aa58d10832b9/d425906b-e7ab-4d10-bbf9-3571bc43ff5e"
-					(reference "U_HALL1")
-					(unit 1)
-				)
-			)
+	(sheet_instances
+		(path "/868f8289-8434-4465-b2f4-2accc5e40bab/3b2478ec-2890-4ec8-b56f-d58b64ce58ab"
+			(page "1")
 		)
 	)
+	(embedded_fonts no)
 )

Commit message: cleanup: annotations and library updates
This is just a task to update the kicad libraries and annotations internally to get that clean ERC.
Parts:
- renumbered C_HALL to C_HALL1, U_HALL to U_HALL1
Changed lines of the file:
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@@
 (kicad_sch
 	(version 20250114)
-	(generator "kicaddy")
-	(generator_version "0.1.0")
+	(generator "eeschema")
+	(generator_version "9.0")
 	(paper "A4")
+	(global_label "GND"
+		(shape passive)
+		(at 166.37 116.84 270)
+		(fields_autoplaced yes)
+		(effects
+			(font
+				(size 1.27 1.27)
+			)
+			(justify right)
+		)
+		(property "Intersheetrefs" "${INTERSHEET_REFS}"
+			(at 166.37 116.84 0)
+			(effects
+				(font
+					(size 1.27 1.27)
+				)
+				(hide yes)
+			)
+		)
+	)
 	(global_label "3V3"
 		(shape passive)
-		(at 128.27 86.36 270)
-		(fields_autoplaced yes)
-		(effects (font (size 1.27 1.27)) (justify left))
+		(at 166.37 109.22 90)
+		(fields_autoplaced yes)
+		(effects
+			(font
+				(size 1.27 1.27)
+			)
+			(justify left)
+		)
+		(property "Intersheetrefs" "${INTERSHEET_REFS}"
+			(at 166.37 109.22 0)
+			(effects
+				(font
+					(size 1.27 1.27)
+				)
+				(hide yes)
+			)
+		)
+	)
+	(global_label "GND"
+		(shape passive)
+		(at 128.27 106.68 270)
+		(fields_autoplaced yes)
+		(effects
+			(font
+				(size 1.27 1.27)
+			)
+			(justify right)
+		)
+		(property "Intersheetrefs" "${INTERSHEET_REFS}"
+			(at 128.27 106.68 0)
+			(effects
+				(font
+					(size 1.27 1.27)
+				)
+				(hide yes)
+			)
+		)
 	)
 	(global_label "3V3"
 		(shape passive)
-		(at 166.37 109.22 270)
-		(fields_autoplaced yes)
-		(effects (font (size 1.27 1.27)) (justify left))
-	)
-	(global_label "GND"
-		(shape passive)
-		(at 128.27 106.68 90)
-		(fields_autoplaced yes)
-		(effects (font (size 1.27 1.27)) (justify right))
-	)
-	(global_label "GND"
-		(shape passive)
-		(at 166.37 116.84 90)
-		(fields_autoplaced yes)
-		(effects (font (size 1.27 1.27)) (justify right))
+		(at 128.27 86.36 90)
+		(fields_autoplaced yes)
+		(effects
+			(font
+				(size 1.27 1.27)
+			)
+			(justify left)
+		)
+		(property "Intersheetrefs" "${INTERSHEET_REFS}"
+			(at 128.27 86.36 0)
+			(effects
+				(font
+					(size 1.27 1.27)
+				)
+				(hide yes)
+			)
+		)
 	)
 	(hierarchical_label "TRIG_ANALOG"
 		(shape output)
-		(at 138.43 96.52 180)
+		(at 138.43 96.52 0)
+		(effects
+			(font
+				(size 1.27 1.27)
+			)
+			(justify left)
+		)
+	)
+	(symbol
+		(lib_id "Device:C")
+		(at 166.37 113.03 0)
+		(unit 1)
+		(exclude_from_sim no)
+		(in_bom yes)
+		(on_board yes)
+		(dnp no)
+		(fields_autoplaced yes)
+		(property "Reference" "C_HALL1"
+			(at 167.005 115.57 0)
+			(effects
+				(font
+					(size 1.27 1.27)
+				)
+				(justify left)
+			)
+		)
+		(property "Value" "100nF"
+			(at 167.005 110.49 0)
+			(effects
+				(font
+					(size 1.27 1.27)
+				)
+				(justify left)
+			)
+		)
+		(property "Footprint" "Capacitor_SMD:C_0402_1005Metric"
+			(at 167.3352 109.22 0)
+			(effects
+				(font
+					(size 1.27 1.27)
+				)
+				(hide yes)
+			)
+		)
+		(property "Datasheet" "~"
+			(at 166.37 113.03 0)
+			(effects
+				(font
+					(size 1.27 1.27)
+				)
+				(hide yes)
+			)
+		)
+		(property "Description" "Unpolarized capacitor"
+			(at 166.37 113.03 0)
+			(effects
+				(font
+					(size 1.27 1.27)
+				)
+				(hide yes)
+			)
+		)
+		(pin "1"
+		)
+		(pin "2"
+		)
+		(instances
+			(project "snips_controller"
+				(path "/868f8289-8434-4465-b2f4-2accc5e40bab/3b2478ec-2890-4ec8-b56f-d58b64ce58ab"
+					(reference "C_HALL1")
+					(unit 1)
+				)
+			)
+		)
 	)
 	(symbol
@@
 		(dnp no)
 		(fields_autoplaced yes)
-		(property "Reference"
-			"U_HALL"
+		(property "Reference" "U_HALL1"
 			(at 135.89 109.22 0)
-			(effects (font (size 1.27 1.27)))
-		)
-		(property "Value"
-			"DRV5055A2"
+			(effects
+				(font
+					(size 1.27 1.27)
+				)
+			)
+		)
+		(property "Value" "DRV5055A2"
 			(at 138.43 106.68 0)
-			(effects (font (size 1.27 1.27)))
-		)
-		(property "Footprint"
-			"Package_TO_SOT_THT:TO-92_Inline"
+			(effects
+				(font
+					(size 1.27 1.27)
+				)
+			)
+		)
+		(property "Footprint" "Package_TO_SOT_THT:TO-92_Inline"
 			(at 130.81 96.52 0)
-			(effects (font (size 1.27 1.27)) (hide yes))
-		)
-		(property "Datasheet"
-			"https://www.ti.com/lit/ds/symlink/drv5055-q1.pdf"
+			(effects
+				(font
+					(size 1.27 1.27)
+				)
+				(hide yes)
+			)
+		)
+		(property "Datasheet" "https://www.ti.com/lit/ds/symlink/drv5055-q1.pdf"
 			(at 130.81 96.52 0)
-			(effects (font (size 1.27 1.27)) (hide yes))
-		)
-		(property "Description"
-			"50 mV/mT,±42-mT, 20-kHz, 3.3/5V, TO-92"
+			(effects
+				(font
+					(size 1.27 1.27)
+				)
+				(hide yes)
+			)
+		)
+		(property "Description" "50 mV/mT,±42-mT, 20-kHz, 3.3/5V, TO-92"
 			(at 130.81 96.52 0)
-			(effects (font (size 1.27 1.27)) (hide yes))
-		)
-		(pin "1")
-		(pin "2")
-		(pin "3")
+			(effects
+				(font
+					(size 1.27 1.27)
+				)
+				(hide yes)
+			)
+		)
+		(pin "1"
+		)
+		(pin "2"
+		)
+		(pin "3"
+		)
 		(instances
-			(project ""
+			(project "snips_controller"
 				(path "/868f8289-8434-4465-b2f4-2accc5e40bab/3b2478ec-2890-4ec8-b56f-d58b64ce58ab"
-					(reference "U_HALL")
+					(reference "U_HALL1")
 					(unit 1)
 				)
@@
 		)
 	)
-	(symbol
-		(lib_id "Device:C")
-		(at 166.37 113.03 0)
-		(unit 1)
-		(exclude_from_sim no)
-		(in_bom yes)
-		(on_board yes)
-		(dnp no)
-		(fields_autoplaced yes)
-		(property "Reference"
-			"C_HALL"
-			(at 167.005 115.57 0)
-			(effects (font (size 1.27 1.27)) (justify left))
-		)
-		(property "Value"
-			"100nF"
-			(at 167.005 110.49 0)
-			(effects (font (size 1.27 1.27)) (justify left))
-		)
-		(property "Footprint"
-			"Capacitor_SMD:C_0402_1005Metric"
-			(at 167.3352 109.22 0)
-			(effects (font (size 1.27 1.27)) (hide yes))
-		)
-		(property "Datasheet"
-			"~"
-			(at 166.37 113.03 0)
-			(effects (font (size 1.27 1.27)) (hide yes))
-		)
-		(property "Description"
-			"Unpolarized capacitor"
-			(at 166.37 113.03 0)
-			(effects (font (size 1.27 1.27)) (hide yes))
-		)
-		(pin "1")
-		(pin "2")
-		(instances
-			(project ""
-				(path "/868f8289-8434-4465-b2f4-2accc5e40bab/3b2478ec-2890-4ec8-b56f-d58b64ce58ab"
-					(reference "C_HALL")
-					(unit 1)
-				)
-			)
-		)
-	)
-	(sheet_instances
-		(path "/868f8289-8434-4465-b2f4-2accc5e40bab/3b2478ec-2890-4ec8-b56f-d58b64ce58ab"
-			(page "1")
-		)
-	)
-	(embedded_fonts no)
 )
