File: PCB/oled.kicad_sch (KiCad schematic)
At the start: 5 parts

Commit message: refactor: erc is clean
This gets the schematic as clean as it can be.
Parts:
- removed R_I2C_SCL, R_I2C_SDA: 4.7kΩ, symbol Device:R
- removed U_OLED: SSD1306_1.3in, symbol SnipsControllers:SSD1306_OLED_4pin
- added R_I2C_SCL1, R_I2C_SDA1: 4.7kΩ, symbol Device:R
- added U_OLED1: SSD1306_1.3in, symbol SnipsControllers:SSD1306_OLED_4pin
Connections:
- net 3V3: now also R_I2C_SCL1.1, R_I2C_SDA1.1, U_OLED1.1 (VCC)
- net GND: now also U_OLED1.2 (GND)
- net I2C_SCL: now also R_I2C_SCL1.2, U_OLED1.3 (SCL)
- net I2C_SDA: now also R_I2C_SDA1.2, U_OLED1.4 (SDA)

Commit message: refactor: switch over to esp32-s3-wroom1 (#13)
This refactors to the esp32-s3 to avoid every problem we encountered with the raspberry pi options.
Parts:
- removed R_I2C_SCL1, R_I2C_SDA1: 4.7kΩ, symbol Device:R
- removed U_OLED1: SSD1306_1.3in, symbol SnipsControllers:SSD1306_OLED_4pin
- added R_I2C_SCL, R_I2C_SDA: 4.7kΩ, Resistor_SMD:R_0402_1005Metric, symbol Device:R
- added U_OLED: SSD1306_1.3in, Display:Adafruit_SSD1306, symbol SnipsControllers:SSD1306_OLED_4pin
- C_OLED_1: footprint (none) -> Capacitor_SMD:C_0805_2012Metric
- C_OLED_2: footprint (none) -> Capacitor_SMD:C_0402_1005Metric
Connections:
- net 3V3: now also R_I2C_SCL.1, R_I2C_SDA.1, U_OLED.1 (VCC)
- net GND: now also U_OLED.2 (GND)
- net I2C_SCL: now also R_I2C_SCL.2, U_OLED.3 (SCL)
- net I2C_SDA: now also R_I2C_SDA.2, U_OLED.4 (SDA)

Commit message: cleanup: annotations and library updates
This is just a task to update the kicad libraries and annotations internally to get that clean ERC.
Parts:
- renumbered R_I2C_SCL to R_I2C_SCL1, R_I2C_SDA to R_I2C_SDA1, U_OLED to U_OLED1
