File: PCB/oled.kicad_sch (KiCad schematic)
At the start: 3 parts

Commit message: task: write matched LCSC part numbers into the schematic
Adds scripts/apply_lcsc_fields.py, which clones each symbol's existing
Manufacturer_Part_Number property (same indentation/effects) into a new
'LCSC' field with the matched code -- the field name the Fabrication
Toolkit plugin already installed in this repo recognizes for JLCPCB BOM
matching.

Applied the 31 confirmed matches from jlc_match.py across all sheets
(68 individual references). C_BUCK_OUT1 and R_ISET1 are left without an
LCSC field -- JLC doesn't stock those exact Yageo part numbers, to be
sorted out separately.

Verified: kicad-cli sch export bom round-trips every LCSC value
correctly, and ERC reports 0 violations.

Also switched jlc_match.py's BOM export to unranged references so each
match maps cleanly to individual schematic symbols.

Co-Authored-By: Claude Sonnet 5 <noreply@anthropic.com>
Parts:
- C_OLED_1: LCSC (none) -> C2982567
- C_OLED_2: LCSC (none) -> C131394
- U_OLED1: LCSC (none) -> C160404
Changed lines of the file:
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@@
+			)
+		)
+		(property "LCSC" "C160404"
+			(at 0 0 0)
+			(hide yes)
+			(show_name no)
+			(do_not_autoplace no)
+			(effects
+				(font
+					(size 1.27 1.27)
+				)
 			)
 		)
@@
 			)
 		)
+		(property "LCSC" "C2982567"
+			(at 0 0 0)
+			(hide yes)
+			(show_name no)
+			(do_not_autoplace no)
+			(effects
+				(font
+					(size 1.27 1.27)
+				)
+			)
+		)
 		(pin "1"
 		)
@@
 			(at 0 0 0)
 			(hide yes)
+			(show_name no)
+			(do_not_autoplace no)
+			(effects
+				(font
+					(size 1.27 1.27)
+				)
+			)
+		)
+		(property "LCSC" "C131394"
+			(at 0 0 0)
+			(hide yes)
