File: PCB/snips_controller.kicad_sch (KiCad schematic)
At the start: 94 parts, among them X1 12MHz

Commit message: refactor: break apart schematic into sub sheets
This breaks apart the main schematic file into 14 sub sheets that are easier to maintain.
Parts:
- removed BT1: Li-ion_18650_or_14500, symbol Device:Battery
- removed C16, C17: 15pF, symbol Device:C
- removed C_1V1_1, C_1V1_2, C_ADC_AVDD1, C_DBNC, C_HALL, C_IOVDD_1, C_IOVDD_2, C_OLED_2, C_QSPI_IOVDD, C_RGB, C_STICK, C_SYS_2, C_VIN_2, C_XBEE_RC, C_XBEE_VCC: 100nF, symbol Device:C
- removed C_ADC_AVDD2, C_VREG_1, C_VREG_2, C_VREG_AVDD, C_WL_VBAT1, C_WL_VBAT2: 4.7µF, symbol Device:C
- removed C_BAT, C_BUCK_IN, C_OLED_1, C_SYS_1, C_VIN_1: 10µF, symbol Device:C
- removed C_BUCK_OUT: 22µF, symbol Device:C
- removed C_WL_VIO: 2.2µF, symbol Device:C
- removed D_MACRO1, D_MACRO2, D_MACRO3, D_MACRO4, D_MACRO5, D_MACRO6: 1N4148, symbol Device:D_Small
- removed D_OR1, D_OR2: 1N4148W, symbol Device:D_Small
- removed D_RGB: SK6812, LED_SMD:LED_SK6812_PLCC4_5.0x5.0mm_P3.2mm, symbol LED:SK6812
- removed J_STICK: GuliKit_Thumbstick, symbol Connector_Generic:Conn_01x05
- removed J_USB: USB-C, symbol Connector:USB_C_Receptacle_USB2.0_16P
- removed L_BUCK: 1µH, symbol Device:L
- removed L_VREG: 3.3µH, symbol Device:L
- removed L_WL_VBAT: 2.2µH, symbol Device:L
- removed Q_LATCH: 2N7002, symbol Transistor_FET:Q_NMOS_GSD
- removed Q_PWR: DMG2305UX, symbol Transistor_FET:Q_PMOS_GSD
- removed R11: 1kΩ, symbol Device:R
- removed R22: 470Ω, symbol Device:R
- removed R23, R_LATCH_G, R_STAT1, R_TS, R_XBEE_RST: 10kΩ, symbol Device:R
- removed R_ADC_AVDD1: 200Ω, symbol Device:R
- removed R_ADC_AVDD2: 1Ω, symbol Device:R
- removed R_BTN_PU, R_FB1, R_GATE, R_PWR_SENSE, R_VSYS2: 100kΩ, symbol Device:R
- removed R_CC1, R_CC2: 5.1kΩ, symbol Device:R
- removed R_FB2: 56.2kΩ, symbol Device:R
- removed R_I2C_SCL, R_I2C_SDA: 4.7kΩ, symbol Device:R
- removed R_ISET: 600Ω, symbol Device:R
- removed R_RGB: 330Ω, symbol Device:R
- removed R_USB_DM, R_USB_DP: 27Ω, symbol Device:R
- removed R_VSET: 18kΩ, symbol Device:R
- removed R_VSYS1: 200kΩ, symbol Device:R
- removed R_XBEE_RC: 100Ω, symbol Device:R
- removed SW_BOOTSEL: TP-1221U-K9K5325, symbol Switch:SW_Push
- removed SW_MACRO1, SW_MACRO2, SW_MACRO3, SW_MACRO4, SW_MACRO5, SW_MACRO6, SW_PWR, SW_TRIG_DIG, SW_VOL_DN, SW_VOL_UP: Omron_B3F, symbol Switch:SW_Push
- removed U_BUCK: TLV62569, Package_TO_SOT_SMD:SOT-23-5, symbol Regulator_Switching:TLV62569DBV
- removed U_CHG: bq25185, BQ25185DLHR:IC_BQ25185DLHR, symbol BQ25185DLHR:BQ25185DLHR
- removed U_FLASH: W25Q32RVXHJQ, Package_SO:SOIC-8_5.3x5.3mm_P1.27mm, symbol Memory_Flash:W25Q32JVSS
- removed U_HALL: DRV5055A2, Package_TO_SOT_THT:TO-92_Inline, symbol Sensor_Magnetic:DRV5055A2xLPGxQ1
- removed U_LPO: 32.768kHz_oscillator, symbol SnipsControllers:Osc_32k768_3pin
- removed U_MCU: RP2350A0A2, Package_DFN_QFN:QFN-60-1EP_7x7mm_P0.4mm_EP3.4x3.4mm, symbol MCU_RaspberryPi:RP2350A
- removed U_OLED: SSD1306_1.3in, symbol SnipsControllers:SSD1306_OLED_4pin
- removed U_WIFI: LBEE5KL1YN, symbol SnipsControllers:Murata_Type1YN
- removed U_XBEE: XBee3, XB324Z8UTJ, symbol Xbee3:XB3-24Z8UT-J
- removed X1: 12MHz, symbol Device:Crystal
Other:
- added sheet Battery (battery.kicad_sch)
- added sheet Button_Matrix (button_matrix.kicad_sch)
- added sheet Buttons_Direct (buttons_direct.kicad_sch)
- added sheet Hall_Trigger (hall_trigger.kicad_sch)
- added sheet MCU_Core (mcu_core.kicad_sch)
- added sheet OLED (oled.kicad_sch)
- added sheet Power_Buck (power_buck.kicad_sch)
- added sheet Power_Charger (power_charger.kicad_sch)
- added sheet Power_Control (power_control.kicad_sch)
- added sheet RGB_LED (rgb_led.kicad_sch)
- added sheet Thumbstick (thumbstick.kicad_sch)
- added sheet USB_C (usb_c.kicad_sch)
- added sheet Wireless (wireless.kicad_sch)
- added sheet XBee (xbee.kicad_sch)

Commit message: refactor: switch over to esp32-s3-wroom1 (#13)
This refactors to the esp32-s3 to avoid every problem we encountered with the raspberry pi options.
Other:
- removed sheet Button_Matrix
- removed sheet Wireless
- sheet Buttons_Direct ports: added BTN_MACRO1, BTN_MACRO2, BTN_MACRO3, BTN_MACRO4, BTN_MACRO5, BTN_MACRO6; removed none
- sheet MCU_Core ports: added BTN_MACRO1, BTN_MACRO2, BTN_MACRO3, BTN_MACRO4, BTN_MACRO5, BTN_MACRO6, PWR_BTN_SENSE; removed GP15_SENSE, MAT_C0, MAT_C1, MAT_C2, MAT_R0, MAT_R1, WL_CLK, WL_CS, WL_D, WL_ON
- sheet Power_Control ports: added PWR_BTN_SENSE; removed GP15_SENSE
