File: PCB/snips_controller.kicad_sch (KiCad schematic)
At the start: 0 parts

Commit message: refactor: swap footprints and add symmetry
This updates the footprints of a couple components to be smaller and closer to what we want. It also adds two buttons to ensure left and right side symmetry.
Other:
- sheet Buttons_Direct ports: added BTN_THR_DN, BTN_THR_UP; removed none
- sheet MCU_Core ports: added BTN_THR_DN, BTN_THR_UP; removed none

Commit message: task: generate production files (#27)
* task: generate production files

We have wrapped up board validation. Gerbers are now generated. Logo generated. Good to go.

* refactor: added STAT2

It was worth adding and will give us more info during battery charging.
Other:
- sheet MCU_Core ports: added STAT2; removed none
- sheet Power_Charger ports: added STAT2; removed none
Changed lines of the file:
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@@
+	(wire
+		(pts
+			(xy 905.51 350.52) (xy 515.62 199.39)
+		)
+		(stroke
+			(width 0)
+			(type default)
+		)
+	)
 	(wire
 		(pts
@@
 			)
 		)
+		(pin "STAT2" input
+			(at 905.51 350.52 90)
+			(effects
+				(font
+					(size 1.27 1.27)
+				)
+				(justify right)
+			)
+		)
 		(pin "PWR_BTN_SENSE" bidirectional
 			(at 934.72 350.52 90)
@@
 			(effects
 				(font
+					(size 1.27 1.27)
+				)
+				(justify right)
+			)
+		)
+		(pin "STAT2" output
+			(at 515.62 199.39 270)
+			(effects
+				(font
