File: PCB/snips_controller.kicad_sch (KiCad schematic)
At the start: 0 parts

Commit message: Accelerometer-driven low-power mode (hardware, PCB only) (#47)
* feat: accelerometer-driven low-power mode (hardware, PCB 1/2)

Adds a QMA6100P accelerometer (I2C, shared OLED bus) and enables
host-commanded XBee pin-sleep, laying the hardware groundwork for a
low-power mode: OLED off + XBee sleep after a short idle timeout (no
buttons, no motion), full soft-latch power-off after a longer one.

- QMA6100P chosen after checking JLCPCB's actual parts library: no
  candidate accelerometer is Basic-library, so it won on price, size,
  and standby current (500nA), which matters since it has to watch for
  motion through the whole low-power period.
- Hand-authored symbol + footprint (no existing library part) — pad
  geometry pulled from JLCPCB/LCSC's own EasyEDA component data
  (LCSC C2887190), not estimated from the datasheet's low-res drawing.
- New Accelerometer sheet, wired into the existing I2C bus and into a
  new GPIO46 (INT1) interrupt line so the MCU can light-sleep instead
  of polling for wake conditions.
- XBee DTR moved off its permanent GND tie onto GPIO42 (SLEEP_RQ), so
  firmware can actually request/cancel pin-sleep instead of the radio
  being forced awake at all times.
- Placed, routed, DRC- and ERC-clean.

Firmware (driver, low-power state machine) and production file
generation are follow-up work — this PR is hardware/schematic only.

Co-Authored-By: Claude Sonnet 5 <noreply@anthropic.com>

* feat: accelerometer-driven low-power mode (firmware, PCB 2/2)

Progressive-enhancement low-power mode: idle cascade through
full -> dim OLED -> OLED off -> XBee sleep (each stage independently
timed, capped by a configurable aggressiveness mode), plus an
independent auto-poweroff timer that fires regardless of mode.

- PowerManager (power_management.h/.cpp): pure, unit-tested state
  machine. Takes "did anything happen this tick" and current time,
  reports which tier to be in and a one-shot poweroff flag. No
  capability flags needed for progressive enhancemen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
Other:
- added sheet Accelerometer (accelerometer.kicad_sch)
Changed lines of the file:
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@@
 	(generator_version "10.0")
 	(paper "A4")
+	(junction
+		(at 982.98 849.63)
+		(diameter 0)
+		(color 0 0 0 0)
+	)
+	(junction
+		(at 949.96 849.63)
+		(diameter 0)
+		(color 0 0 0 0)
+	)
 	(wire
 		(pts
@@
 	(wire
 		(pts
+			(xy 905.51 350.52) (xy 515.62 199.39)
+		)
+		(stroke
+			(width 0)
+			(type default)
+		)
+	)
+	(wire
+		(pts
 			(xy 1883.41 999.49) (xy 1247.14 849.63)
 		)
@@
 	(wire
 		(pts
+			(xy 217.17 999.49) (xy 982.98 849.63)
+		)
+		(stroke
+			(width 0)
+			(type default)
+		)
+	)
+	(wire
+		(pts
+			(xy 82.55 999.49) (xy 949.96 849.63)
+		)
+		(stroke
+			(width 0)
+			(type default)
+		)
+	)
+	(wire
+		(pts
 			(xy 1807.21 999.49) (xy 1181.1 849.63)
 		)
@@
 		(pts
 			(xy 877.57 350.52) (xy 500.38 199.39)
-		)
-		(stroke
-			(width 0)
-			(type default)
-		)
-	)
-	(wire
-		(pts
-			(xy 905.51 350.52) (xy 515.62 199.39)
 		)
 		(stroke
@@
 				)
 			)
+		)
+	)
+	(sheet
+		(at 0 999.49)
+		(size 299.72 200.66)
+		(exclude_from_sim no)
+		(in_bom yes)
+		(on_board yes)
+		(dnp no)
+		(stroke
+			(width 0.1524)
+			(type solid)
+		)
+		(fill
+			(color 0 0 0 0)
+		)
+		(property "Sheetname" "Accelerometer"
+			(at 0 998.7784 0)
+			(show_name no)
+			(do_not_autoplace no)
+			(effects
+				(font
+					(size 1.27 1.27)
+				)
+				(justify left bottom)
+			)
+		)
+		(property "Sheetfile" "accelerometer.kicad_sch"
+			(at 0 1200.7346 0)
+			(show_name no)
+			(do_not_autoplace no)
+			(effects
+				(font
+					(size 1.27 1.27)
+				)
+				(justify left top)
+			)
+		)
+		(pin "I2C_SDA" bidirectional
+			(at 82.55 999.49 90)
+			(effects
+				(font
+					(size 1.27 1.27)
+				)
+				(justify right)
+			)
+		)
+		(pin "I2C_SCL" bidirectional
+			(at 217.17 999.49 90)
+			(effects
+				(font
+					(size 1.27 1.27)
+				)
+				(justify right)
+			)
+		)
+		(instances
+			(project "snips_controller"
+				(path "/21935953-32a0-46ad-8079-8177920c6978"
+					(page "14")
+				)
+			)
