File: PCB/power_charger.kicad_sch (KiCad schematic)
At the start: 10 parts

Commit message: task: generate production files (#27)
* task: generate production files

We have wrapped up board validation. Gerbers are now generated. Logo generated. Good to go.

* refactor: added STAT2

It was worth adding and will give us more info during battery charging.
Parts:
- added R_STAT2: 10kΩ, Resistor_SMD:R_0402_1005Metric, symbol Device:R
Connections:
- net 3V3: now also R_STAT2.2
- net STAT2: now reaches U_CHG1.3 (STAT2)
- net STAT2: now also R_STAT2.1
