File: PCB/power_charger.kicad_sch (KiCad schematic)
At the start: 11 parts

Commit message: task: write matched LCSC part numbers into the schematic
Adds scripts/apply_lcsc_fields.py, which clones each symbol's existing
Manufacturer_Part_Number property (same indentation/effects) into a new
'LCSC' field with the matched code -- the field name the Fabrication
Toolkit plugin already installed in this repo recognizes for JLCPCB BOM
matching.

Applied the 31 confirmed matches from jlc_match.py across all sheets
(68 individual references). C_BUCK_OUT1 and R_ISET1 are left without an
LCSC field -- JLC doesn't stock those exact Yageo part numbers, to be
sorted out separately.

Verified: kicad-cli sch export bom round-trips every LCSC value
correctly, and ERC reports 0 violations.

Also switched jlc_match.py's BOM export to unranged references so each
match maps cleanly to individual schematic symbols.

Co-Authored-By: Claude Sonnet 5 <noreply@anthropic.com>
Parts:
- C_BAT1, C_SYS_1, C_VIN_1: LCSC (none) -> C2982567
- C_SYS_2, C_VIN_2: LCSC (none) -> C131394
- R_STAT1, R_STAT2, R_TS1: LCSC (none) -> C60490
- R_VSET1: LCSC (none) -> C138044
- U_CHG1: LCSC (none) -> C19725033
Changed lines of the file:
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@@
+			)
+		)
+		(property "LCSC" "C138044"
+			(at 0 0 0)
+			(hide yes)
+			(show_name no)
+			(do_not_autoplace no)
+			(effects
+				(font
+					(size 1.27 1.27)
+				)
 			)
 		)
@@
 			)
 		)
+		(property "LCSC" "C131394"
+			(at 0 0 0)
+			(hide yes)
+			(show_name no)
+			(do_not_autoplace no)
+			(effects
+				(font
+					(size 1.27 1.27)
+				)
+			)
+		)
 		(pin "1"
 		)
@@
 			)
 		)
+		(property "LCSC" "C60490"
+			(at 0 0 0)
+			(hide yes)
+			(show_name no)
+			(do_not_autoplace no)
+			(effects
+				(font
+					(size 1.27 1.27)
+				)
+			)
+		)
 		(pin "1"
 		)
@@
 			)
 		)
+		(property "LCSC" "C60490"
+			(at 0 0 0)
+			(hide yes)
+			(show_name no)
+			(do_not_autoplace no)
+			(effects
+				(font
+					(size 1.27 1.27)
+				)
+			)
+		)
 		(pin "1"
 		)
@@
 			)
 		)
+		(property "LCSC" "C2982567"
+			(at 0 0 0)
+			(hide yes)
+			(show_name no)
+			(do_not_autoplace no)
+			(effects
+				(font
+					(size 1.27 1.27)
+				)
+			)
+		)
 		(pin "1"
 		)
@@
 			)
 		)
+		(property "LCSC" "C19725033"
+			(at 0 0 0)
+			(hide yes)
+			(show_name no)
+			(do_not_autoplace no)
+			(effects
+				(font
+					(size 1.27 1.27)
+				)
+			)
+		)
 		(pin "1"
 		)
@@
 			)
 		)
+		(property "LCSC" "C2982567"
+			(at 0 0 0)
+			(hide yes)
+			(show_name no)
+			(do_not_autoplace no)
+			(effects
+				(font
+					(size 1.27 1.27)
+				)
+			)
+		)
 		(pin "1"
 		)
@@
 			)
 		)
+		(property "LCSC" "C131394"
+			(at 0 0 0)
+			(hide yes)
+			(show_name no)
+			(do_not_autoplace no)
+			(effects
+				(font
+					(size 1.27 1.27)
+				)
+			)
+		)
 		(pin "1"
 		)
@@
 			)
 		)
+		(property "LCSC" "C2982567"
+			(at 0 0 0)
+			(hide yes)
+			(show_name no)
+			(do_not_autoplace no)
+			(effects
+				(font
+					(size 1.27 1.27)
+				)
+			)
+		)
 		(pin "1"
 		)
@@
 			(at 0 0 0)
 			(hide yes)
+			(show_name no)
+			(do_not_autoplace no)
+			(effects
+				(font
+					(size 1.27 1.27)
+				)
+			)
+		)
+		(property "LCSC" "C60490"
+			(at 0 0 0)
+			(hide yes)

Commit message: fix: swap the 2 JLC-unstocked parts for equivalents
C_BUCK_OUT1: same 22uF/0805/X5R/16V/10% spec, just TDK
(C2012X5R1C226KT000E) instead of Yageo -- JLC doesn't carry that exact
Yageo part number, TDK's is otherwise identical and well stocked.

R_ISET1: 600R isn't a standard E96 value, so no manufacturer stocks a
0402 chip resistor at that exact resistance -- confirmed via an
exhaustive JLC catalog search (package-filtered, zero real resistor
hits). Moved to 604R, the nearest E96 value (0.67% off, inside the
part's own 1% tolerance band), same Yageo family
(AC0402FR-07604RL). This is the charge-current-set resistor on the
bq25185; a 0.67% shift in set current is negligible.

Both now carry LCSC fields (C76637, C227167) -- all 33 BOM parts are
now matched. Verified via kicad-cli sch export bom and sch erc (0
violations).

Co-Authored-By: Claude Sonnet 5 <noreply@anthropic.com>
Parts:
- R_ISET1: value 600Ω -> 604Ω; LCSC (none) -> C227167; Manufacturer_Part_Number RC0402FR-07600RL -> AC0402FR-07604RL
Changed lines of the file:
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@@
 			)
 		)
-		(property "Value" "600Ω"
+		(property "Value" "604Ω"
 			(at 148.59 92.71 90)
 			(show_name no)
@@
 			)
 		)
-		(property "Manufacturer_Part_Number" "RC0402FR-07600RL"
+		(property "Manufacturer_Part_Number" "AC0402FR-07604RL"
 			(at 0 0 0)
 			(hide yes)
+			(show_name no)
+			(do_not_autoplace no)
+			(effects
+				(font
+					(size 1.27 1.27)
+				)
+			)
+		)
+		(property "LCSC" "C227167"
+			(at 0 0 0)
+			(hide yes)
