File: PCB/power_charger.kicad_sch (KiCad schematic)
At the start: 11 parts

Commit message: task: add JLCPCB/LCSC part-matching script (#31)
* task: add JLCPCB/LCSC part-matching script

Looks up every BOM line's Manufacturer + MPN (fields every part in this
project already carries) against JLCPCB's public component-search
endpoint -- the same one jlcpcb.com's own search box uses, no API key
needed -- and reports the matched LCSC part number.

Report-only for now: it doesn't touch the schematic. 31/33 parts on the
board matched automatically in testing; the 2 misses (C_BUCK_OUT1,
R_ISET1) genuinely aren't in JLC's catalog under those exact Yageo part
numbers, confirmed by zero search results, not a matching bug.

Co-Authored-By: Claude Sonnet 5 <noreply@anthropic.com>

* task: write matched LCSC part numbers into the schematic

Adds scripts/apply_lcsc_fields.py, which clones each symbol's existing
Manufacturer_Part_Number property (same indentation/effects) into a new
'LCSC' field with the matched code -- the field name the Fabrication
Toolkit plugin already installed in this repo recognizes for JLCPCB BOM
matching.

Applied the 31 confirmed matches from jlc_match.py across all sheets
(68 individual references). C_BUCK_OUT1 and R_ISET1 are left without an
LCSC field -- JLC doesn't stock those exact Yageo part numbers, to be
sorted out separately.

Verified: kicad-cli sch export bom round-trips every LCSC value
correctly, and ERC reports 0 violations.

Also switched jlc_match.py's BOM export to unranged references so each
match maps cleanly to individual schematic symbols.

Co-Authored-By: Claude Sonnet 5 <noreply@anthropic.com>

* fix: swap the 2 JLC-unstocked parts for equivalents

C_BUCK_OUT1: same 22uF/0805/X5R/16V/10% spec, just TDK
(C2012X5R1C226KT000E) instead of Yageo -- JLC doesn't carry that exact
Yageo part number, TDK's is otherwise identical and well stocked.

R_ISET1: 600R isn't a standard E96 value, so no manufacturer stocks a
0402 chip resistor at that exact resistance -- confirmed via an
exhaustive JLC catalog search (package-filtered, zero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
Parts:
- C_BAT1, C_SYS_1, C_VIN_1: LCSC (none) -> C2982567
- C_SYS_2, C_VIN_2: LCSC (none) -> C131394
- R_ISET1: value 600Ω -> 604Ω; LCSC (none) -> C227167; Manufacturer_Part_Number RC0402FR-07600RL -> AC0402FR-07604RL
- R_STAT1, R_STAT2, R_TS1: LCSC (none) -> C60490
- R_VSET1: LCSC (none) -> C138044
- U_CHG1: LCSC (none) -> C19725033
Changed lines of the file:
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@@
+			)
+		)
+		(property "LCSC" "C138044"
+			(at 0 0 0)
+			(hide yes)
+			(show_name no)
+			(do_not_autoplace no)
+			(effects
+				(font
+					(size 1.27 1.27)
+				)
 			)
 		)
@@
 			)
 		)
+		(property "LCSC" "C131394"
+			(at 0 0 0)
+			(hide yes)
+			(show_name no)
+			(do_not_autoplace no)
+			(effects
+				(font
+					(size 1.27 1.27)
+				)
+			)
+		)
 		(pin "1"
 		)
@@
 			)
 		)
+		(property "LCSC" "C60490"
+			(at 0 0 0)
+			(hide yes)
+			(show_name no)
+			(do_not_autoplace no)
+			(effects
+				(font
+					(size 1.27 1.27)
+				)
+			)
+		)
 		(pin "1"
 		)
@@
 			)
 		)
+		(property "LCSC" "C60490"
+			(at 0 0 0)
+			(hide yes)
+			(show_name no)
+			(do_not_autoplace no)
+			(effects
+				(font
+					(size 1.27 1.27)
+				)
+			)
+		)
 		(pin "1"
 		)
@@
 			)
 		)
+		(property "LCSC" "C2982567"
+			(at 0 0 0)
+			(hide yes)
+			(show_name no)
+			(do_not_autoplace no)
+			(effects
+				(font
+					(size 1.27 1.27)
+				)
+			)
+		)
 		(pin "1"
 		)
@@
 			)
 		)
+		(property "LCSC" "C19725033"
+			(at 0 0 0)
+			(hide yes)
+			(show_name no)
+			(do_not_autoplace no)
+			(effects
+				(font
+					(size 1.27 1.27)
+				)
+			)
+		)
 		(pin "1"
 		)
@@
 			)
 		)
+		(property "LCSC" "C2982567"
+			(at 0 0 0)
+			(hide yes)
+			(show_name no)
+			(do_not_autoplace no)
+			(effects
+				(font
+					(size 1.27 1.27)
+				)
+			)
+		)
 		(pin "1"
 		)
@@
 			)
 		)
+		(property "LCSC" "C131394"
+			(at 0 0 0)
+			(hide yes)
+			(show_name no)
+			(do_not_autoplace no)
+			(effects
+				(font
+					(size 1.27 1.27)
+				)
+			)
+		)
 		(pin "1"
 		)
@@
 			)
 		)
-		(property "Value" "600Ω"
+		(property "Value" "604Ω"
 			(at 148.59 92.71 90)
 			(show_name no)
@@
 			)
 		)
-		(property "Manufacturer_Part_Number" "RC0402FR-07600RL"
+		(property "Manufacturer_Part_Number" "AC0402FR-07604RL"
+			(at 0 0 0)
+			(hide yes)
+			(show_name no)
+			(do_not_autoplace no)
+			(effects
+				(font
+					(size 1.27 1.27)
+				)
+			)
+		)
+		(property "LCSC" "C227167"
 			(at 0 0 0)
 			(hide yes)
@@
 			)
 		)
+		(property "LCSC" "C2982567"
+			(at 0 0 0)
+			(hide yes)
+			(show_name no)
+			(do_not_autoplace no)
+			(effects
+				(font
+					(size 1.27 1.27)
+				)
+			)
+		)
 		(pin "1"
 		)
@@
 			(at 0 0 0)
 			(hide yes)
+			(show_name no)
+			(do_not_autoplace no)
+			(effects
+				(font
+					(size 1.27 1.27)
+				)
+			)
+		)
+		(property "LCSC" "C60490"
+			(at 0 0 0)
+			(hide yes)

Commit message: fix: swap 3 JLCPCB-out-of-stock parts for in-stock equivalents
C_BAT1/C_BUCK_IN1/C_OLED_1/C_SYS_1/C_VIN_1 (10uF 0805 X5R 16V):
Yageo CC0805KRX5R7BB106 was at 0 stock -> HRE CGA0805X5R106K160MT
(LCSC C6119886, stock ~254k). Identical spec, different brand.

D_VBUS_TVS1: Nexperia PESD5V0S1BA,115 was down to 1 in stock -> TECH
PUBLIC TPPESD5V0S1BA (LCSC C587144, stock ~981k), a widely-stocked
pin/spec-compatible clone of the same part, same SOD-323 package.

Q_PWR1: Diodes Inc DMG2305UX-7 was down to 8 in stock -> Diodes Inc
DMG2305UX-13 (LCSC C144153, stock ~25k) -- same manufacturer, same
part, the -7/-13 suffix is just reel size (7"/13"), not an electrical
variant.

Found via live JLCPCB stock lookups after the JLCPCB upload flagged
these 3 with shortfalls. Verified via kicad-cli sch export bom and
sch erc (0 violations).

Note: PCB/snips_controller.kicad_pcb and the production/ exports still
need another Update-PCB-from-Schematic + Fabrication Toolkit pass to
pick up these changes -- not included here since they're a separate
manual step (see kicad_pcb_sync_gotcha note).

Co-Authored-By: Claude Sonnet 5 <noreply@anthropic.com>
Parts:
- C_BAT1, C_SYS_1, C_VIN_1: LCSC C2982567 -> C6119886; MF Yageo -> HRE; Manufacturer_Part_Number CC0805KRX5R7BB106 -> CGA0805X5R106K160MT
Changed lines of the file:
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@@
 			)
 		)
-		(property "MF" "Yageo"
-			(at 0 0 0)
-			(hide yes)
-			(show_name no)
-			(do_not_autoplace no)
-			(effects
-				(font
-					(size 1.27 1.27)
-				)
-			)
-		)
-		(property "Manufacturer_Part_Number" "CC0805KRX5R7BB106"
-			(at 0 0 0)
-			(hide yes)
-			(show_name no)
-			(do_not_autoplace no)
-			(effects
-				(font
-					(size 1.27 1.27)
-				)
-			)
-		)
-		(property "LCSC" "C2982567"
+		(property "MF" "HRE"
+			(at 0 0 0)
+			(hide yes)
+			(show_name no)
+			(do_not_autoplace no)
+			(effects
+				(font
+					(size 1.27 1.27)
+				)
+			)
+		)
+		(property "Manufacturer_Part_Number" "CGA0805X5R106K160MT"
+			(at 0 0 0)
+			(hide yes)
+			(show_name no)
+			(do_not_autoplace no)
+			(effects
+				(font
+					(size 1.27 1.27)
+				)
+			)
+		)
+		(property "LCSC" "C6119886"
 			(at 0 0 0)
 			(hide yes)
@@
 			)
 		)
-		(property "MF" "Yageo"
-			(at 0 0 0)
-			(hide yes)
-			(show_name no)
-			(do_not_autoplace no)
-			(effects
-				(font
-					(size 1.27 1.27)
-				)
-			)
-		)
-		(property "Manufacturer_Part_Number" "CC0805KRX5R7BB106"
-			(at 0 0 0)
-			(hide yes)
-			(show_name no)
-			(do_not_autoplace no)
-			(effects
-				(font
-					(size 1.27 1.27)
-				)
-			)
-		)
-		(property "LCSC" "C2982567"
+		(property "MF" "HRE"
+			(at 0 0 0)
+			(hide yes)
+			(show_name no)
+			(do_not_autoplace no)
+			(effects
+				(font
+					(size 1.27 1.27)
+				)
+			)
+		)
+		(property "Manufacturer_Part_Number" "CGA0805X5R106K160MT"
+			(at 0 0 0)
+			(hide yes)
+			(show_name no)
+			(do_not_autoplace no)
+			(effects
+				(font
+					(size 1.27 1.27)
+				)
+			)
+		)
+		(property "LCSC" "C6119886"
 			(at 0 0 0)
 			(hide yes)
@@
 			)
 		)
-		(property "MF" "Yageo"
-			(at 0 0 0)
-			(hide yes)
-			(show_name no)
-			(do_not_autoplace no)
-			(effects
-				(font
-					(size 1.27 1.27)
-				)
-			)
-		)
-		(property "Manufacturer_Part_Number" "CC0805KRX5R7BB106"
-			(at 0 0 0)
-			(hide yes)
-			(show_name no)
-			(do_not_autoplace no)
-			(effects
-				(font
-					(size 1.27 1.27)
-				)
-			)
-		)
-		(property "LCSC" "C2982567"
-			(at 0 0 0)
-			(hide yes)
+		(property "MF" "HRE"
+			(at 0 0 0)
+			(hide yes)
+			(show_name no)
+			(do_not_autoplace no)
+			(effects
+				(font
+					(size 1.27 1.27)
+				)
+			)
+		)
+		(property "Manufacturer_Part_Number" "CGA0805X5R106K160MT"
+			(at 0 0 0)
+			(hide yes)
+			(show_name no)
+			(do_not_autoplace no)
+			(effects
+				(font
+					(size 1.27 1.27)
+				)
+			)
+		)
+		(property "LCSC" "C6119886"
+			(at 0 0 0)
+			(hide yes)
