File: PCB/power_buck.kicad_sch (KiCad schematic)
At the start: 6 parts

Commit message: task: add JLCPCB/LCSC part-matching script (#31)
* task: add JLCPCB/LCSC part-matching script

Looks up every BOM line's Manufacturer + MPN (fields every part in this
project already carries) against JLCPCB's public component-search
endpoint -- the same one jlcpcb.com's own search box uses, no API key
needed -- and reports the matched LCSC part number.

Report-only for now: it doesn't touch the schematic. 31/33 parts on the
board matched automatically in testing; the 2 misses (C_BUCK_OUT1,
R_ISET1) genuinely aren't in JLC's catalog under those exact Yageo part
numbers, confirmed by zero search results, not a matching bug.

Co-Authored-By: Claude Sonnet 5 <noreply@anthropic.com>

* task: write matched LCSC part numbers into the schematic

Adds scripts/apply_lcsc_fields.py, which clones each symbol's existing
Manufacturer_Part_Number property (same indentation/effects) into a new
'LCSC' field with the matched code -- the field name the Fabrication
Toolkit plugin already installed in this repo recognizes for JLCPCB BOM
matching.

Applied the 31 confirmed matches from jlc_match.py across all sheets
(68 individual references). C_BUCK_OUT1 and R_ISET1 are left without an
LCSC field -- JLC doesn't stock those exact Yageo part numbers, to be
sorted out separately.

Verified: kicad-cli sch export bom round-trips every LCSC value
correctly, and ERC reports 0 violations.

Also switched jlc_match.py's BOM export to unranged references so each
match maps cleanly to individual schematic symbols.

Co-Authored-By: Claude Sonnet 5 <noreply@anthropic.com>

* fix: swap the 2 JLC-unstocked parts for equivalents

C_BUCK_OUT1: same 22uF/0805/X5R/16V/10% spec, just TDK
(C2012X5R1C226KT000E) instead of Yageo -- JLC doesn't carry that exact
Yageo part number, TDK's is otherwise identical and well stocked.

R_ISET1: 600R isn't a standard E96 value, so no manufacturer stocks a
0402 chip resistor at that exact resistance -- confirmed via an
exhaustive JLC catalog search (package-filtered, zero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
Parts:
- C_BUCK_IN1: LCSC (none) -> C2982567
- C_BUCK_OUT1: LCSC (none) -> C76637; MF Yageo -> TDK; Manufacturer_Part_Number CC0805KRX5R7BB226 -> C2012X5R1C226KT000E
- L_BUCK1: LCSC (none) -> C913207
- R_FB1: LCSC (none) -> C327361
- R_FB2: LCSC (none) -> C183355
- U_BUCK1: LCSC (none) -> C141836
Changed lines of the file:
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@@
+			)
+		)
+		(property "LCSC" "C327361"
+			(at 0 0 0)
+			(hide yes)
+			(show_name no)
+			(do_not_autoplace no)
+			(effects
+				(font
+					(size 1.27 1.27)
+				)
 			)
 		)
@@
 			)
 		)
+		(property "LCSC" "C913207"
+			(at 0 0 0)
+			(hide yes)
+			(show_name no)
+			(do_not_autoplace no)
+			(effects
+				(font
+					(size 1.27 1.27)
+				)
+			)
+		)
 		(pin "1"
 		)
@@
 			)
 		)
+		(property "LCSC" "C141836"
+			(at 0 0 0)
+			(hide yes)
+			(show_name no)
+			(do_not_autoplace no)
+			(effects
+				(font
+					(size 1.27 1.27)
+				)
+			)
+		)
 		(pin "1"
 		)
@@
 			)
 		)
+		(property "LCSC" "C2982567"
+			(at 0 0 0)
+			(hide yes)
+			(show_name no)
+			(do_not_autoplace no)
+			(effects
+				(font
+					(size 1.27 1.27)
+				)
+			)
+		)
 		(pin "1"
 		)
@@
 			)
 		)
-		(property "MF" "Yageo"
-			(at 0 0 0)
-			(hide yes)
-			(show_name no)
-			(do_not_autoplace no)
-			(effects
-				(font
-					(size 1.27 1.27)
-				)
-			)
-		)
-		(property "Manufacturer_Part_Number" "CC0805KRX5R7BB226"
+		(property "MF" "TDK"
+			(at 0 0 0)
+			(hide yes)
+			(show_name no)
+			(do_not_autoplace no)
+			(effects
+				(font
+					(size 1.27 1.27)
+				)
+			)
+		)
+		(property "Manufacturer_Part_Number" "C2012X5R1C226KT000E"
+			(at 0 0 0)
+			(hide yes)
+			(show_name no)
+			(do_not_autoplace no)
+			(effects
+				(font
+					(size 1.27 1.27)
+				)
+			)
+		)
+		(property "LCSC" "C76637"
 			(at 0 0 0)
 			(hide yes)
@@
 			(at 0 0 0)
 			(hide yes)
+			(show_name no)
+			(do_not_autoplace no)
+			(effects
+				(font
+					(size 1.27 1.27)
+				)
+			)
+		)
+		(property "LCSC" "C183355"
+			(at 0 0 0)
+			(hide yes)
