File: PCB/usb_c.kicad_sch (KiCad schematic)
At the start: 4 parts

Commit message: task: write matched LCSC part numbers into the schematic
Adds scripts/apply_lcsc_fields.py, which clones each symbol's existing
Manufacturer_Part_Number property (same indentation/effects) into a new
'LCSC' field with the matched code -- the field name the Fabrication
Toolkit plugin already installed in this repo recognizes for JLCPCB BOM
matching.

Applied the 31 confirmed matches from jlc_match.py across all sheets
(68 individual references). C_BUCK_OUT1 and R_ISET1 are left without an
LCSC field -- JLC doesn't stock those exact Yageo part numbers, to be
sorted out separately.

Verified: kicad-cli sch export bom round-trips every LCSC value
correctly, and ERC reports 0 violations.

Also switched jlc_match.py's BOM export to unranged references so each
match maps cleanly to individual schematic symbols.

Co-Authored-By: Claude Sonnet 5 <noreply@anthropic.com>
Parts:
- D_VBUS_TVS1: LCSC (none) -> C19224
- J_USB1: LCSC (none) -> C165948
- R_CC1, R_CC2: LCSC (none) -> C105872
Changed lines of the file:
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@@
+			)
+		)
+		(property "LCSC" "C165948"
+			(at 0 0 0)
+			(hide yes)
+			(show_name no)
+			(do_not_autoplace no)
+			(effects
+				(font
+					(size 1.27 1.27)
+				)
 			)
 		)
@@
 			)
 		)
+		(property "LCSC" "C105872"
+			(at 0 0 0)
+			(hide yes)
+			(show_name no)
+			(do_not_autoplace no)
+			(effects
+				(font
+					(size 1.27 1.27)
+				)
+			)
+		)
 		(pin "1"
 		)
@@
 			)
 		)
+		(property "LCSC" "C105872"
+			(at 0 0 0)
+			(hide yes)
+			(show_name no)
+			(do_not_autoplace no)
+			(effects
+				(font
+					(size 1.27 1.27)
+				)
+			)
+		)
 		(pin "1"
 		)
@@
 			(at 0 0 0)
 			(hide yes)
+			(show_name no)
+			(do_not_autoplace no)
+			(effects
+				(font
+					(size 1.27 1.27)
+				)
+			)
+		)
+		(property "LCSC" "C19224"
+			(at 0 0 0)
+			(hide yes)

Commit message: fix: swap 3 JLCPCB-out-of-stock parts for in-stock equivalents
C_BAT1/C_BUCK_IN1/C_OLED_1/C_SYS_1/C_VIN_1 (10uF 0805 X5R 16V):
Yageo CC0805KRX5R7BB106 was at 0 stock -> HRE CGA0805X5R106K160MT
(LCSC C6119886, stock ~254k). Identical spec, different brand.

D_VBUS_TVS1: Nexperia PESD5V0S1BA,115 was down to 1 in stock -> TECH
PUBLIC TPPESD5V0S1BA (LCSC C587144, stock ~981k), a widely-stocked
pin/spec-compatible clone of the same part, same SOD-323 package.

Q_PWR1: Diodes Inc DMG2305UX-7 was down to 8 in stock -> Diodes Inc
DMG2305UX-13 (LCSC C144153, stock ~25k) -- same manufacturer, same
part, the -7/-13 suffix is just reel size (7"/13"), not an electrical
variant.

Found via live JLCPCB stock lookups after the JLCPCB upload flagged
these 3 with shortfalls. Verified via kicad-cli sch export bom and
sch erc (0 violations).

Note: PCB/snips_controller.kicad_pcb and the production/ exports still
need another Update-PCB-from-Schematic + Fabrication Toolkit pass to
pick up these changes -- not included here since they're a separate
manual step (see kicad_pcb_sync_gotcha note).

Co-Authored-By: Claude Sonnet 5 <noreply@anthropic.com>
Parts:
- D_VBUS_TVS1: LCSC C19224 -> C587144; MF Nexperia -> TECH PUBLIC; Manufacturer_Part_Number PESD5V0S1BA,115 -> TPPESD5V0S1BA
Changed lines of the file:
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@@
 			)
 		)
-		(property "MF" "Nexperia"
+		(property "MF" "TECH PUBLIC"
 			(at 0 0 0)
 			(hide yes)
@@
 			)
 		)
-		(property "Manufacturer_Part_Number" "PESD5V0S1BA,115"
+		(property "Manufacturer_Part_Number" "TPPESD5V0S1BA"
 			(at 0 0 0)
 			(hide yes)
@@
 			)
 		)
-		(property "LCSC" "C19224"
+		(property "LCSC" "C587144"
 			(at 0 0 0)
 			(hide yes)
