File: PCB/rgb_led.kicad_sch (KiCad schematic)
At the start: 3 parts

Commit message: task: write matched LCSC part numbers into the schematic
Adds scripts/apply_lcsc_fields.py, which clones each symbol's existing
Manufacturer_Part_Number property (same indentation/effects) into a new
'LCSC' field with the matched code -- the field name the Fabrication
Toolkit plugin already installed in this repo recognizes for JLCPCB BOM
matching.

Applied the 31 confirmed matches from jlc_match.py across all sheets
(68 individual references). C_BUCK_OUT1 and R_ISET1 are left without an
LCSC field -- JLC doesn't stock those exact Yageo part numbers, to be
sorted out separately.

Verified: kicad-cli sch export bom round-trips every LCSC value
correctly, and ERC reports 0 violations.

Also switched jlc_match.py's BOM export to unranged references so each
match maps cleanly to individual schematic symbols.

Co-Authored-By: Claude Sonnet 5 <noreply@anthropic.com>
Parts:
- C_RGB1: LCSC (none) -> C131394
- D_RGB1: LCSC (none) -> C5149201
- R_RGB1: LCSC (none) -> C105875
Changed lines of the file:
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@@
+			)
+		)
+		(property "LCSC" "C131394"
+			(at 0 0 0)
+			(hide yes)
+			(show_name no)
+			(do_not_autoplace no)
+			(effects
+				(font
+					(size 1.27 1.27)
+				)
 			)
 		)
@@
 			)
 		)
+		(property "LCSC" "C105875"
+			(at 0 0 0)
+			(hide yes)
+			(show_name no)
+			(do_not_autoplace no)
+			(effects
+				(font
+					(size 1.27 1.27)
+				)
+			)
+		)
 		(pin "1"
 		)
@@
 			(at 0 0 0)
 			(hide yes)
+			(show_name no)
+			(do_not_autoplace no)
+			(effects
+				(font
+					(size 1.27 1.27)
+				)
+			)
+		)
+		(property "LCSC" "C5149201"
+			(at 0 0 0)
+			(hide yes)

Commit message: task: swap 13 Extended-library parts for Basic-library equivalents
Swaps 39 individual references (13 unique parts) from JLC's Extended
library to verified Basic-library equivalents, to cut the per-part
setup/handling fee that made our first JLCPCB quote ($333.84) come in
well above PCBWay's (~$190):

- 6 capacitor values (10uF/0603, 100nF/0402, 10uF/0805, 22uF/0805,
  1uF/0603, 47pF/0402) -> Samsung Electro-Mechanics / FH, same
  value+package, tolerance/voltage equal or better.
- 4 resistor values (10k/100k/5.1k/200k, all 0402 +-1%) -> UNI-ROYAL,
  identical spec.
- 1N4148W (D_OR1/D_OR2) and 2N7002 (Q_LATCH1) -> different brands of
  the same industry-standard generic part, same footprint.
- R_XBEE_RC1 (100R/0402) -> UNI-ROYAL 0402WGF1000TCE (C25076), found
  by manual search after the tool's automated keyword search missed
  it in its top-25 results -- a known search-relevance gap, not a
  wrong match (verified directly against JLC's listing).

Verified via kicad-cli sch export bom (all 33 BOM rows correct) and
sch erc (0 violations).

Note: same as prior schematic-only PRs, PCB/snips_controller.kicad_pcb
and production/ exports still need another Update-PCB-from-Schematic +
Fabrication Toolkit pass before re-uploading anywhere.

Co-Authored-By: Claude Sonnet 5 <noreply@anthropic.com>
Parts:
- C_RGB1: LCSC C131394 -> C1525; MF Yageo -> Samsung Electro-Mechanics; Manufacturer_Part_Number CC0402KRX7R9BB104 -> CL05B104KO5NNNC
Changed lines of the file:
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@@
 			)
 		)
-		(property "MF" "Yageo"
+		(property "MF" "Samsung Electro-Mechanics"
 			(at 0 0 0)
 			(hide yes)
@@
 			)
 		)
-		(property "Manufacturer_Part_Number" "CC0402KRX7R9BB104"
+		(property "Manufacturer_Part_Number" "CL05B104KO5NNNC"
 			(at 0 0 0)
 			(hide yes)
@@
 			)
 		)
-		(property "LCSC" "C131394"
+		(property "LCSC" "C1525"
 			(at 0 0 0)
 			(hide yes)
