File: PCB/thumbstick.kicad_sch (KiCad schematic)
At the start: 2 parts

Commit message: task: write matched LCSC part numbers into the schematic
Adds scripts/apply_lcsc_fields.py, which clones each symbol's existing
Manufacturer_Part_Number property (same indentation/effects) into a new
'LCSC' field with the matched code -- the field name the Fabrication
Toolkit plugin already installed in this repo recognizes for JLCPCB BOM
matching.

Applied the 31 confirmed matches from jlc_match.py across all sheets
(68 individual references). C_BUCK_OUT1 and R_ISET1 are left without an
LCSC field -- JLC doesn't stock those exact Yageo part numbers, to be
sorted out separately.

Verified: kicad-cli sch export bom round-trips every LCSC value
correctly, and ERC reports 0 violations.

Also switched jlc_match.py's BOM export to unranged references so each
match maps cleanly to individual schematic symbols.

Co-Authored-By: Claude Sonnet 5 <noreply@anthropic.com>
Parts:
- C_STICK1: LCSC (none) -> C131394
Changed lines of the file:
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@@
+			)
+		)
+		(property "LCSC" "C131394"
+			(at 0 0 0)
+			(hide yes)
+			(show_name no)
+			(do_not_autoplace no)
+			(effects
+				(font
+					(size 1.27 1.27)
+				)
 			)
 		)

Commit message: task: alert on Basic-library alternatives during JLC part matching (#33)
* task: alert on Basic-library alternatives during JLC part matching

JLC's "Extended" library carries a per-unique-part setup fee on top of
unit price; "Basic" doesn't. That fee doesn't amortize well on a board
with many distinct low-quantity parts -- confirmed the hard way: our
first real JLCPCB assembly quote came back at $333.84 vs PCBWay's
~$190 for the same order, and all 33 of our matched parts were
Extended.

jlc_match.py now does a secondary search for a same-value/same-package
Basic-library part whenever the real match lands on Extended, and
flags it in the report (new BasicAlt column + a Status alert) rather
than silently leaving it. On the current board this surfaces 11
plausible Basic-library swaps (common resistor/cap values, and the
generic 1N4148W diode and 2N7002 MOSFET, which are industry-standard
parts many brands stock identically).

This is alert-only, same as the rest of this script -- it doesn't
touch the schematic. Spot-checked 4 of the 11 suggestions directly
against JLC's catalog to confirm value/package actually match, not
just a keyword hit.

Co-Authored-By: Claude Sonnet 5 <noreply@anthropic.com>

* fix: two correctness bugs in Basic-library alternative matching

1. find_basic_alternative() trusted the raw keyword-search hit without
   verifying the candidate's actual value -- JLC's fuzzy full-text search
   can return a wrong-value part that just shares digits (e.g. searching
   "100 0402" surfaced a 1kΩ resistor, EIA code "1001", as a false match
   for a 100Ω part). Now parses and compares the actual numeric value
   (with unit) before accepting a candidate; falls back to exact
   model-name matching for non-numeric values (generic diode/transistor
   part families like "1N4148W", "2N7002").

2. The new value parser's regex required the unit to be the first
   character of the string, but JLC resistor descriptions carry a
   Chinese prefix ("厚膜电阻 10kΩ ±1%" = "thi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
Parts:
- C_STICK1: LCSC C131394 -> C1525; MF Yageo -> Samsung Electro-Mechanics; Manufacturer_Part_Number CC0402KRX7R9BB104 -> CL05B104KO5NNNC
Changed lines of the file:
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@@
 			)
 		)
-		(property "MF" "Yageo"
+		(property "MF" "Samsung Electro-Mechanics"
 			(at 0 0 0)
 			(hide yes)
@@
 			)
 		)
-		(property "Manufacturer_Part_Number" "CC0402KRX7R9BB104"
+		(property "Manufacturer_Part_Number" "CL05B104KO5NNNC"
 			(at 0 0 0)
 			(hide yes)
@@
 			)
 		)
-		(property "LCSC" "C131394"
+		(property "LCSC" "C1525"
 			(at 0 0 0)
 			(hide yes)
