File: PCB/thumbstick.kicad_sch (KiCad schematic)
At the start: 2 parts

Commit message: fix: make every BOM Value unambiguous for the fab, and switch D_INV_ISO1 to SOT-323 (#61)
* fix: make every BOM Value unambiguous for the fab, and switch D_INV_ISO1 to SOT-323

PCBWay flagged D_INV_ISO1: "BAT54W" is SOT-323 from nearly every maker, but we
had picked Yangjie's SOD-123 variant. A fab only sees Designator, Footprint,
Quantity and Value in the BOM (never MF/MPN/LCSC), so a bare part name is
ambiguous. Fixes the class of problem, not just this part:

- Every component's Value is now "<label> | <MPN> | <manufacturer> | <package>"
  (label dropped when it repeats the MPN; commas/periods stripped so the CSV
  never needs quoting). BT1 keeps its RIGHT-ANGLE HORIZONTAL note. Applied to
  all 81 parts across every sheet and the PCB.
- scripts/bom_values.py builds, applies, and checks these values, including
  that the PCB copy of Value/MF/MPN/footprint matches the schematic. New
  footprints must be added to its package table on purpose; hand-sourced parts
  with no MPN (J_STICK1) are listed explicitly.
- D_INV_ISO1 -> Diodes BAT54W-7-F in SOT-323 (common part, several makers).
  Pin 1 anode / pin 2 not connected / pin 3 cathode, confirmed against
  Nexperia's numbered pinning table and Diodes' datasheet. Uses KiCad's
  Diode:BAT54W symbol; PCB footprint replaced and rerouted. Electrically the
  same BAT54 family (30V, 200mA, 2uA leakage at 25V), so the SPICE model and
  scripts/spice/latch_sim.py still pass.
- Layout diagrams now say AO3401A for Q_PWR1 (they were stale since it was
  swapped from DMG2305UX) and BAT54W-7-F/SOT-323 for D_INV_ISO1.
- Repo CLAUDE.md documents the Value rule and the script.

ERC/DRC clean; production files regenerated.

Co-Authored-By: Claude Sonnet 5 <noreply@anthropic.com>

* chore: commit KiCad project settings (reordered used-designators list)

Co-Authored-By: Claude Sonnet 5 <noreply@anthropic.com>

---------

Co-authored-by: Claude Sonnet 5 <noreply@anthropic.com>
Parts:
- C_STICK1: value 100nF -> 100nF | CL05B104KO5NNNC | Samsung Electro-Mechanics | 0402
Changed lines of the file:
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@@
 			)
 		)
-		(property "Value" "100nF"
+		(property "Value" "100nF | CL05B104KO5NNNC | Samsung Electro-Mechanics | 0402"
 			(at 128.905 101.6 0)
 			(show_name no)
