File: PCB/v2.x/snips_controller.kicad_pcb (KiCad board)
At the start: 4 copper layers, 30 x 70 mm, 94 parts

Commit message: V2 PCB: raise C_LATCH_FB1 to 1 uF for more power-off margin
The XBee carrier takes the 3V3 rail from about 36 uF to about 47 uF
nominal. A heavier rail collapses more slowly, so RXD0's returning
pull-up has longer to act, and with 470 nF the worst-case power-off
margin fell to about 0.03 V.

Use the 1 uF 50 V 0603 already on the board. It raises the worst-case
margin to 0.34 V with the carrier and 0.46 V without it, on the same
pads, and removes a BOM line. Turn-on and power-off get slightly slower.

Run the V2 latch simulation at the carrier's rail, the harder case.

Co-Authored-By: Claude Opus 5.5 <noreply@anthropic.com>
Parts:
- C_LATCH_FB1: value 470nF 25V X7R ±10% | CL10B474KA8NNNC | Samsung | 0603 -> 1µF 50V X5R ±10% | CL10A105KB8NNNC | Samsung | 0603
Changed lines of the file:
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@@
 			)
 		)
-		(property "Stackup Source" "PCB/v2.x/stackup/board.kdl:86"
+		(property "Stackup Source" "PCB/v2.x/stackup/board.kdl:87"
 			(at 0 2 0)
 			(layer "F.SilkS")
@@
 			)
 		)
-		(property "Stackup Source" "PCB/v2.x/stackup/board.kdl:82"
+		(property "Stackup Source" "PCB/v2.x/stackup/board.kdl:83"
 			(at -2 0 0)
 			(layer "F.SilkS")
@@
 			)
 		)
-		(property "Stackup Source" "PCB/v2.x/stackup/board.kdl:112"
+		(property "Stackup Source" "PCB/v2.x/stackup/board.kdl:113"
 			(at 0 2 90)
 			(layer "F.SilkS")
@@
 			)
 		)
-		(property "Stackup Source" "PCB/v2.x/stackup/board.kdl:84"
+		(property "Stackup Source" "PCB/v2.x/stackup/board.kdl:85"
 			(at 0 2 0)
 			(layer "F.SilkS")
@@
 			)
 		)
-		(property "Stackup Source" "PCB/v2.x/stackup/board.kdl:77"
+		(property "Stackup Source" "PCB/v2.x/stackup/board.kdl:78"
 			(at 0 2 90)
 			(layer "F.SilkS")
@@
 			)
 		)
-		(property "Stackup Source" "PCB/v2.x/stackup/board.kdl:91"
+		(property "Stackup Source" "PCB/v2.x/stackup/board.kdl:92"
 			(at 2 0 0)
 			(layer "F.SilkS")
@@
 			)
 		)
-		(property "Stackup Source" "PCB/v2.x/stackup/board.kdl:88"
+		(property "Stackup Source" "PCB/v2.x/stackup/board.kdl:89"
 			(at 0 2 0)
 			(layer "F.SilkS")
@@
 			)
 		)
-		(property "Stackup Source" "PCB/v2.x/stackup/board.kdl:85"
+		(property "Stackup Source" "PCB/v2.x/stackup/board.kdl:86"
 			(at 0 2 0)
 			(layer "F.SilkS")
@@
 			)
 		)
-		(property "Stackup Source" "PCB/v2.x/stackup/board.kdl:83"
+		(property "Stackup Source" "PCB/v2.x/stackup/board.kdl:84"
 			(at 0 2 0)
 			(layer "F.SilkS")
@@
 			)
 		)
-		(property "Stackup Source" "PCB/v2.x/stackup/board.kdl:115"
+		(property "Stackup Source" "PCB/v2.x/stackup/board.kdl:116"
 			(at 0 2 0)
 			(layer "F.SilkS")
@@
 			)
 		)
-		(property "Stackup Source" "PCB/v2.x/stackup/board.kdl:104"
+		(property "Stackup Source" "PCB/v2.x/stackup/board.kdl:105"
 			(at 0 -2 90)
 			(layer "F.SilkS")
@@
 			)
 		)
-		(property "Stackup Source" "PCB/v2.x/stackup/board.kdl:93"
+		(property "Stackup Source" "PCB/v2.x/stackup/board.kdl:94"
 			(at -2 0 0)
 			(layer "F.SilkS")
@@
 			)
 		)
-		(property "Stackup Source" "PCB/v2.x/stackup/board.kdl:73"
+		(property "Stackup Source" "PCB/v2.x/stackup/board.kdl:74"
 			(at -2 0 0)
 			(layer "F.SilkS")
@@
 			)
 		)
-		(property "Stackup Source" "PCB/v2.x/stackup/board.kdl:80"
+		(property "Stackup Source" "PCB/v2.x/stackup/board.kdl:81"
 			(at 0 2 90)
 			(layer "F.SilkS")
@@
 			)
 		)
-		(property "Stackup Source" "PCB/v2.x/stackup/board.kdl:109"
+		(property "Stackup Source" "PCB/v2.x/stackup/board.kdl:110"
 			(at 0 2 90)
 			(layer "F.SilkS")
@@
 			)
 		)
-		(property "Stackup Source" "PCB/v2.x/stackup/board.kdl:90"
+		(property "Stackup Source" "PCB/v2.x/stackup/board.kdl:91"
 			(at 2 0 0)
 			(layer "F.SilkS")
@@
 			)
 		)
-		(property "Stackup Source" "PCB/v2.x/stackup/board.kdl:108"
+		(property "Stackup Source" "PCB/v2.x/stackup/board.kdl:109"
 			(at 0 2 90)
 			(layer "F.SilkS")
@@
 			)
 		)
-		(property "Stackup Source" "PCB/v2.x/stackup/board.kdl:94"
+		(property "Stackup Source" "PCB/v2.x/stackup/board.kdl:95"
 			(at -2 0 0)
 			(layer "F.SilkS")
@@
 			)
 		)
-		(property "Stackup Source" "PCB/v2.x/stackup/board.kdl:81"
+		(property "Stackup Source" "PCB/v2.x/stackup/board.kdl:82"
 			(at 0 -2 0)
 			(layer "F.SilkS")
@@
 			)
 		)
-		(property "Stackup Source" "PCB/v2.x/stackup/board.kdl:89"
+		(property "Stackup Source" "PCB/v2.x/stackup/board.kdl:90"
 			(at 0 2 0)
 			(layer "F.SilkS")
@@
 			)
 		)
-		(property "Stackup Source" "PCB/v2.x/stackup/board.kdl:78"
+		(property "Stackup Source" "PCB/v2.x/stackup/board.kdl:79"
 			(at 0 2 90)
 			(layer "F.SilkS")
@@
 			)
 		)
-		(property "Stackup Source" "PCB/v2.x/stackup/board.kdl:87"
+		(property "Stackup Source" "PCB/v2.x/stackup/board.kdl:88"
 			(at 0 2 0)
 			(layer "F.SilkS")
@@
 			)
 		)
-		(property "Stackup Source" "PCB/v2.x/stackup/board.kdl:114"
+		(property "Stackup Source" "PCB/v2.x/stackup/board.kdl:115"
 			(at 0 -2 90)
 			(layer "B.SilkS")
@@
 			)
 		)
-		(property "Stackup Source" "PCB/v2.x/stackup/board.kdl:68"
+		(property "Stackup Source" "PCB/v2.x/stackup/board.kdl:69"
 			(at 0 -2 0)
 			(layer "B.SilkS")
@@
 			)
 		)
-		(property "Stackup Source" "PCB/v2.x/stackup/board.kdl:92"
+		(property "Stackup Source" "PCB/v2.x/stackup/board.kdl:93"
 			(at 0 2 0)
 			(layer "B.SilkS")
@@
 			)
 		)
-		(property "Stackup Source" "PCB/v2.x/stackup/board.kdl:69"
+		(property "Stackup Source" "PCB/v2.x/stackup/board.kdl:70"
 			(at -2 0 0)
 			(layer "B.SilkS")
@@
 			)
 		)
-		(property "Stackup Source" "PCB/v2.x/stackup/board.kdl:96"
+		(property "Stackup Source" "PCB/v2.x/stackup/board.kdl:97"
 			(at 0 -2 180)
 			(layer "B.SilkS")
@@
 			)
 		)
-		(property "Stackup Source" "PCB/v2.x/stackup/board.kdl:75"
+		(property "Stackup Source" "PCB/v2.x/stackup/board.kdl:76"
 			(at 0 2 180)
 			(layer "B.SilkS")
@@
 			)
 		)
-		(property "Stackup Source" "PCB/v2.x/stackup/board.kdl:71"
+		(property "Stackup Source" "PCB/v2.x/stackup/board.kdl:72"
 			(at -2 0 270)
 			(layer "B.SilkS")
@@
 			)
 		)
-		(property "Stackup Source" "PCB/v2.x/stackup/board.kdl:79"
+		(property "Stackup Source" "PCB/v2.x/stackup/board.kdl:80"
 			(at 0 -2 180)
 			(layer "B.SilkS")
@@
 			)
 		)
-		(property "Stackup Source" "PCB/v2.x/stackup/board.kdl:74"
+		(property "Stackup Source" "PCB/v2.x/stackup/board.kdl:75"
 			(at 0 -2 180)
 			(layer "B.SilkS")
@@
 			)
 		)
-		(property "Stackup Source" "PCB/v2.x/stackup/board.kdl:70"
+		(property "Stackup Source" "PCB/v2.x/stackup/board.kdl:71"
 			(at 0 -2 180)
 			(layer "B.SilkS")
@@
 			)
 		)
-		(property "Stackup Source" "PCB/v2.x/stackup/board.kdl:107"
+		(property "Stackup Source" "PCB/v2.x/stackup/board.kdl:108"
 			(at 0 -2 180)
 			(layer "B.SilkS")
@@
 			)
 		)
-		(property "Stackup Source" "PCB/v2.x/stackup/board.kdl:95"
+		(property "Stackup Source" "PCB/v2.x/stackup/board.kdl:96"
 			(at -2 0 180)
 			(layer "B.SilkS")
@@
 			)
 		)
-		(property "Stackup Source" "PCB/v2.x/stackup/board.kdl:113"
+		(property "Stackup Source" "PCB/v2.x/stackup/board.kdl:114"
 			(at 0 -2 180)
 			(layer "B.SilkS")
@@
 			)
 		)
-		(property "Value" "470nF 25V X7R ±10% | CL10B474KA8NNNC | Samsung | 0603"
+		(property "Value" "1µF 50V X5R ±10% | CL10A105KB8NNNC | Samsung | 0603"
 			(at 0 -1.43 0)
 			(layer "B.Fab")
@@
 			)
 		)
-		(property "Voltage" "25V"
+		(property "Voltage" "50V"
 			(at 0 -2 0)
 			(layer "B.SilkS")
@@
 			)
 		)
-		(property "Manufacturer_Part_Number" "CL10B474KA8NNNC"
+		(property "Manufacturer_Part_Number" "CL10A105KB8NNNC"
 			(at 0 -2 0)
 			(layer "B.SilkS")
@@
 			)
 		)
-		(property "LCSC" "C1623"
+		(property "LCSC" "C15849"
 			(at 0 -2 0)
 			(layer "B.SilkS")
@@
 			)
 		)
-		(property "Stackup Source" "PCB/v2.x/stackup/board.kdl:67"
+		(property "Stackup Source" "PCB/v2.x/stackup/board.kdl:68"
 			(at 0 -2 0)
 			(layer "B.SilkS")
@@
 			)
 		)
-		(property "Stackup Source" "PCB/v2.x/stackup/board.kdl:111"
+		(property "Stackup Source" "PCB/v2.x/stackup/board.kdl:112"
 			(at 0 -2 270)
 			(layer "B.SilkS")
@@
 			)
 		)
-		(property "Stackup Source" "PCB/v2.x/stackup/board.kdl:76"
+		(property "Stackup Source" "PCB/v2.x/stackup/board.kdl:77"
 			(at 0 -2 180)
 			(layer "B.SilkS")
